Commit message: urdf work start

File: LBR/urdf/iiwa_r820_DH.xacro (robot description, xacro)
@@ -1,5 +1,5 @@
 <?xml version="1.0" ?>
 <robot name="iiwa_r820" xmlns:xacro="http://wiki.ros.org/xacro">
-  <xacro:include filename="$(find iiwa)/urdf/iiwa_r820_DH_macro.xacro"/>
+  <xacro:include filename="$(find rik)/LBR/urdf/iiwa_r820_DH_macro.xacro"/>
   <xacro:iiwa_r820 prefix=""/>
 </robot>

File: LBR/urdf/iiwa_r820_DH_macro.xacro (robot description, xacro)
@@ -7,5 +7,5 @@
         <origin xyz="0 0 0" rpy="0 0 0" />
         <geometry>
-          <mesh filename="package://iiwa/meshes/iiwa_r820/visual/base_link.dae" />
+          <mesh filename="package://rik/LBR/meshes/iiwa_r820/visual/base_link.dae" />
         </geometry>
       </visual>
@@ -13,5 +13,5 @@
         <origin xyz="0 0 0" rpy="0 0 0" />
         <geometry>
-          <mesh filename="package://iiwa/meshes/iiwa_r820/collision/base_link.stl" />
+          <mesh filename="package://rik/LBR/meshes/iiwa_r820/collision/base_link.stl" />
         </geometry>
       </collision>
@@ -21,5 +21,5 @@
         <origin xyz="0 -0.36 0" rpy="-1.5708 0 0" />
         <geometry>
-          <mesh filename="package://iiwa/meshes/iiwa_r820/visual/link_1.dae" />
+          <mesh filename="package://rik/LBR/meshes/iiwa_r820/visual/link_1.dae" />
         </geometry>
       </visual>
@@ -27,5 +27,5 @@
         <origin xyz="0 -0.36 0" rpy="-1.5708 0 0" />
         <geometry>
-          <mesh filename="package://iiwa/meshes/iiwa_r820/collision/link_1.stl" />
+          <mesh filename="package://rik/LBR/meshes/iiwa_r820/collision/link_1.stl" />
         </geometry>
       </collision>
@@ -35,5 +35,5 @@
         <origin xyz="0 0 0" rpy="0 0 0" />
         <geometry>
-          <mesh filename="package://iiwa/meshes/iiwa_r820/visual/link_2.dae" />
+          <mesh filename="package://rik/LBR/meshes/iiwa_r820/visual/link_2.dae" />
         </geometry>
       </visual>
@@ -41,5 +41,5 @@
         <origin xyz="0 0 0" rpy="0 0 0" />
         <geometry>
-          <mesh filename="package://iiwa/meshes/iiwa_r820/collision/link_2.stl" />
+          <mesh filename="package://rik/LBR/meshes/iiwa_r820/collision/link_2.stl" />
         </geometry>
       </collision>
@@ -49,5 +49,5 @@
         <origin xyz="0 -0.42 0" rpy="-1.5708 0 0" />
         <geometry>
-          <mesh filename="package://iiwa/meshes/iiwa_r820/visual/link_3.dae" />
+          <mesh filename="package://rik/LBR/meshes/iiwa_r820/visual/link_3.dae" />
         </geometry>
       </visual>
@@ -55,5 +55,5 @@
         <origin xyz="0 -0.42 0" rpy="-1.5708 0 0" />
         <geometry>
-          <mesh filename="package://iiwa/meshes/iiwa_r820/collision/link_3.stl" />
+          <mesh filename="package://rik/LBR/meshes/iiwa_r820/collision/link_3.stl" />
         </geometry>
       </collision>
@@ -63,5 +63,5 @@
         <origin xyz="0 0 0" rpy="0 0 0" />
         <geometry>
-          <mesh filename="package://iiwa/meshes/iiwa_r820/visual/link_4.dae" />
+          <mesh filename="package://rik/LBR/meshes/iiwa_r820/visual/link_4.dae" />
         </geometry>
       </visual>
@@ -69,5 +69,5 @@
         <origin xyz="0 0 0" rpy="0 0 0" />
         <geometry>
-          <mesh filename="package://iiwa/meshes/iiwa_r820/collision/link_4.stl" />
+          <mesh filename="package://rik/LBR/meshes/iiwa_r820/collision/link_4.stl" />
         </geometry>
       </collision>
@@ -77,5 +77,5 @@
         <origin xyz="0 -0.4 0" rpy="-1.5708 0 0" />
         <geometry>
-          <mesh filename="package://iiwa/meshes/iiwa_r820/visual/link_5.dae" />
+          <mesh filename="package://rik/LBR/meshes/iiwa_r820/visual/link_5.dae" />
         </geometry>
       </visual>
@@ -83,5 +83,5 @@
         <origin xyz="0 -0.4 0" rpy="-1.5708 0 0" />
         <geometry>
-          <mesh filename="package://iiwa/meshes/iiwa_r820/collision/link_5.stl" />
+          <mesh filename="package://rik/LBR/meshes/iiwa_r820/collision/link_5.stl" />
         </geometry>
       </collision>
@@ -91,5 +91,5 @@
         <origin xyz="0 0 0" rpy="0 0 0" />
         <geometry>
-          <mesh filename="package://iiwa/meshes/iiwa_r820/visual/link_6.dae" />
+          <mesh filename="package://rik/LBR/meshes/iiwa_r820/visual/link_6.dae" />
         </geometry>
       </visual>
@@ -97,5 +97,5 @@
         <origin xyz="0 0 0" rpy="0 0 0" />
         <geometry>
-          <mesh filename="package://iiwa/meshes/iiwa_r820/collision/link_6.stl" />
+          <mesh filename="package://rik/LBR/meshes/iiwa_r820/collision/link_6.stl" />
         </geometry>
       </collision>
@@ -106,5 +106,5 @@
         <origin xyz="0 0 -0.126" rpy="0 0 0" />
         <geometry>
-          <mesh filename="package://iiwa/meshes/iiwa_r820/visual/link_7.dae" />
+          <mesh filename="package://rik/LBR/meshes/iiwa_r820/visual/link_7.dae" />
         </geometry>
       </visual>
@@ -112,5 +112,5 @@
         <origin xyz="0 0 -0.126" rpy="0 0 0" />
         <geometry>
-          <mesh filename="package://iiwa/meshes/iiwa_r820/collision/link_7.stl" />
+          <mesh filename="package://rik/LBR/meshes/iiwa_r820/collision/link_7.stl" />
         </geometry>
       </collision>
@@ -128,5 +128,5 @@
     </joint>
     <joint name="${prefix}iiwa_j2" type="revolute">
-      <origin xyz="-0.00043624 0 0" rpy="-1.5708 0 0" />
+      <origin xyz="0 0 0" rpy="-1.5708 0 0" />
       <parent link="${prefix}iiwa_l1" />
       <child link="${prefix}iiwa_l2" />
