Commit message: add 9-dof testy model

File: LBR/urdf/iiwa_r820_DH_macro.xacro (robot description, xacro)
@@ -19,5 +19,5 @@
     <link name="${prefix}iiwa_l1">
       <visual>
-        <origin xyz="0 -0.36 0" rpy="-1.5708 0 0" />
+        <origin xyz="0 -0.36 0" rpy="-${pi/2} 0 0" />
         <geometry>
           <mesh filename="package://rik/LBR/meshes/iiwa_r820/visual/link_1.dae" />
@@ -25,5 +25,5 @@
       </visual>
       <collision>
-        <origin xyz="0 -0.36 0" rpy="-1.5708 0 0" />
+        <origin xyz="0 -0.36 0" rpy="-${pi/2} 0 0" />
         <geometry>
           <mesh filename="package://rik/LBR/meshes/iiwa_r820/collision/link_1.stl" />
@@ -47,5 +47,5 @@
     <link name="${prefix}iiwa_l3">
       <visual>
-        <origin xyz="0 -0.42 0" rpy="-1.5708 0 0" />
+        <origin xyz="0 -0.42 0" rpy="-${pi/2} 0 0" />
         <geometry>
           <mesh filename="package://rik/LBR/meshes/iiwa_r820/visual/link_3.dae" />
@@ -53,5 +53,5 @@
       </visual>
       <collision>
-        <origin xyz="0 -0.42 0" rpy="-1.5708 0 0" />
+        <origin xyz="0 -0.42 0" rpy="-${pi/2} 0 0" />
         <geometry>
           <mesh filename="package://rik/LBR/meshes/iiwa_r820/collision/link_3.stl" />
@@ -75,5 +75,5 @@
     <link name="${prefix}iiwa_l5">
       <visual>
-        <origin xyz="0 -0.4 0" rpy="-1.5708 0 0" />
+        <origin xyz="0 -0.4 0" rpy="-${pi/2} 0 0" />
         <geometry>
           <mesh filename="package://rik/LBR/meshes/iiwa_r820/visual/link_5.dae" />
@@ -81,5 +81,5 @@
       </visual>
       <collision>
-        <origin xyz="0 -0.4 0" rpy="-1.5708 0 0" />
+        <origin xyz="0 -0.4 0" rpy="-${pi/2} 0 0" />
         <geometry>
           <mesh filename="package://rik/LBR/meshes/iiwa_r820/collision/link_5.stl" />
@@ -121,5 +121,5 @@
     <!-- joint list -->
     <joint name="${prefix}iiwa_j1" type="revolute">
-      <origin xyz="0 0 0.36" rpy="1.5708 0 0" />
+      <origin xyz="0 0 0.36" rpy="${pi/2} 0 0" />
       <parent link="${prefix}iiwa_base_link" />
       <child link="${prefix}iiwa_l1" />
@@ -128,5 +128,5 @@
     </joint>
     <joint name="${prefix}iiwa_j2" type="revolute">
-      <origin xyz="0 0 0" rpy="-1.5708 0 0" />
+      <origin xyz="0 0 0" rpy="-${pi/2} 0 0" />
       <parent link="${prefix}iiwa_l1" />
       <child link="${prefix}iiwa_l2" />
@@ -135,5 +135,5 @@
     </joint>
     <joint name="${prefix}iiwa_j3" type="revolute">
-      <origin xyz="0 0 0.42" rpy="1.5708 0 0" />
+      <origin xyz="0 0 0.42" rpy="${pi/2} 0 0" />
       <parent link="${prefix}iiwa_l2" />
       <child link="${prefix}iiwa_l3" />
@@ -142,5 +142,5 @@
     </joint>
     <joint name="${prefix}iiwa_j4" type="revolute">
-      <origin xyz="0.00043624 0 0" rpy="-1.5708 0 0" />
+      <origin xyz="0.00043624 0 0" rpy="-${pi/2} 0 0" />
       <parent link="${prefix}iiwa_l3" />
       <child link="${prefix}iiwa_l4" />
@@ -149,5 +149,5 @@
     </joint>
     <joint name="${prefix}iiwa_j5" type="revolute">
-      <origin xyz="0 0 0.4" rpy="1.5708 0 0" />
+      <origin xyz="0 0 0.4" rpy="${pi/2} 0 0" />
       <parent link="${prefix}iiwa_l4" />
       <child link="${prefix}iiwa_l5" />
@@ -156,5 +156,5 @@
     </joint>
     <joint name="${prefix}iiwa_j6" type="revolute">
-      <origin xyz="0 0 0" rpy="-1.5708 0 0" />
+      <origin xyz="0 0 0" rpy="-${pi/2} 0 0" />
       <parent link="${prefix}iiwa_l5" />
       <child link="${prefix}iiwa_l6" />
