Commit message: urdf parser strt

File: robots/TESTy/urdf/testy_macro.xacro (robot description, xacro)
@@ -389,5 +389,5 @@
     <!-- ROS testy_base_link to KUKA $ROBROOT coordinate system transform -->
     <link name="base" />
-    <joint name="testy_base_link-base" type="fixed">
+    <joint name="testy_base_link->base" type="fixed">
       <origin xyz="0 0 0" rpy="0 0 0"/>
       <parent link="testy_base_link"/>
@@ -395,5 +395,5 @@
     </joint>
     <link name="base_link" />
-    <joint name="base_link-testy_base_link" type="fixed">
+    <joint name="base_link->testy_base_link" type="fixed">
       <origin xyz="0 0 0" rpy="0 0 0"/>
       <parent link="testy_base_link"/>

Commit message: model create beg

File: robots/TESTy/urdf/testy_macro.xacro (robot description, xacro)
@@ -287,5 +287,5 @@
     </joint>
     <joint name="testy_l1->testy_j2_l" type="revolute">
-      <origin xyz="0 0 0.26" rpy="-${pi/2} 0 0" />
+      <origin xyz="0 0 0.26" rpy="-${pi/2} 0.1 0.3" />
       <parent link="testy_l1" />
       <child link="testy_j2_l" />

Commit message: reasons to rethink an architecture

File: robots/TESTy/urdf/testy_macro.xacro (robot description, xacro)
@@ -287,5 +287,5 @@
     </joint>
     <joint name="testy_l1->testy_j2_l" type="revolute">
-      <origin xyz="0 0 0.26" rpy="-${pi/2} 0.1 0.3" />
+      <origin xyz="0 0 0.26" rpy="-${pi/2} 0 0" />
       <parent link="testy_l1" />
       <child link="testy_j2_l" />
