Commit message: second handy

File: robots/TESTy/urdf/testy_1_macro.xacro (robot description, xacro)
@@ -1,259 +1,259 @@
 <?xml version="1.0"?>
 <robot xmlns:xacro="http://wiki.ros.org/xacro">
-  <xacro:macro name="testy">
+  <xacro:macro name="testy_1">
     <!-- link list -->
-    <link name="testy_base_link">
-      <visual>
-        <origin xyz="0 0 0" rpy="0 0 0" />
-        <geometry>
-          <mesh filename="package://rik/robots/TESTy/meshes/visual/link.dae" />
-        </geometry>
-      </visual>
-      <collision>
-        <origin xyz="0 0 0" rpy="0 0 0" />
-        <geometry>
-          <mesh filename="package://rik/robots/TESTy/meshes/collision/link.stl" />
-        </geometry>
-      </collision>
-    </link>
-    <link name="testy_j1_l">
-      <visual>
-        <origin xyz="0 0 0" rpy="0 0 0" />
-        <geometry>
-          <mesh filename="package://rik/robots/TESTy/meshes/visual/joint.dae" />
-        </geometry>
-      </visual>
-      <collision>
-        <origin xyz="0 0 0" rpy="0 0 0" />
-        <geometry>
-          <mesh filename="package://rik/robots/TESTy/meshes/collision/joint.stl" />
-        </geometry>
-      </collision>
-    </link>
-    <link name="testy_l1">
-      <visual>
-        <origin xyz="0 0 0" rpy="0 0 0" />
-        <geometry>
-          <mesh filename="package://rik/robots/TESTy/meshes/visual/link.dae" />
-        </geometry>
-      </visual>
-      <collision>
-        <origin xyz="0 0 0" rpy="0 0 0" />
-        <geometry>
-          <mesh filename="package://rik/robots/TESTy/meshes/collision/link.stl" />
-        </geometry>
-      </collision>
-    </link>
-    <link name="testy_j2_l">
-      <visual>
-        <origin xyz="0 0 0" rpy="0 0 0" />
-        <geometry>
-          <mesh filename="package://rik/robots/TESTy/meshes/visual/joint.dae" />
-        </geometry>
-      </visual>
-      <collision>
-        <origin xyz="0 0 0" rpy="0 0 0" />
-        <geometry>
-          <mesh filename="package://rik/robots/TESTy/meshes/collision/joint.stl" />
-        </geometry>
-      </collision>
-    </link>
-    <link name="testy_l2">
-      <visual>
-        <origin xyz="0 0 0" rpy="0 0 0" />
-        <geometry>
-          <mesh filename="package://rik/robots/TESTy/meshes/visual/link.dae" />
-        </geometry>
-      </visual>
-      <collision>
-        <origin xyz="0 0 0" rpy="0 0 0" />
-        <geometry>
-          <mesh filename="package://rik/robots/TESTy/meshes/collision/link.stl" />
-        </geometry>
-      </collision>
-    </link>
-    <link name="testy_j3_l">
-      <visual>
-        <origin xyz="0 0 0" rpy="0 0 0" />
-        <geometry>
-          <mesh filename="package://rik/robots/TESTy/meshes/visual/joint.dae" />
-        </geometry>
-      </visual>
-      <collision>
-        <origin xyz="0 0 0" rpy="0 0 0" />
-        <geometry>
-          <mesh filename="package://rik/robots/TESTy/meshes/collision/joint.stl" />
-        </geometry>
-      </collision>
-    </link>
-    <link name="testy_l3">
-      <visual>
-        <origin xyz="0 0 0" rpy="0 0 0" />
-        <geometry>
-          <mesh filename="package://rik/robots/TESTy/meshes/visual/link.dae" />
-        </geometry>
-      </visual>
-      <collision>
-        <origin xyz="0 0 0" rpy="0 0 0" />
-        <geometry>
-          <mesh filename="package://rik/robots/TESTy/meshes/collision/link.stl" />
-        </geometry>
-      </collision>
-    </link>
-    <link name="testy_j4_l">
-      <visual>
-        <origin xyz="0 0 0" rpy="0 0 0" />
-        <geometry>
-          <mesh filename="package://rik/robots/TESTy/meshes/visual/joint.dae" />
-        </geometry>
-      </visual>
-      <collision>
-        <origin xyz="0 0 0" rpy="0 0 0" />
-        <geometry>
-          <mesh filename="package://rik/robots/TESTy/meshes/collision/joint.stl" />
-        </geometry>
-      </collision>
-    </link>
-    <link name="testy_l4">
-      <visual>
-        <origin xyz="0 0 0" rpy="0 0 0" />
-        <geometry>
-          <mesh filename="package://rik/robots/TESTy/meshes/visual/link.dae" />
-        </geometry>
-      </visual>
-      <collision>
-        <origin xyz="0 0 0" rpy="0 0 0" />
-        <geometry>
-          <mesh filename="package://rik/robots/TESTy/meshes/collision/link.stl" />
-        </geometry>
-      </collision>
-    </link>
-    <link name="testy_j5_l">
-      <visual>
-        <origin xyz="0 0 0" rpy="0 0 0" />
-        <geometry>
-          <mesh filename="package://rik/robots/TESTy/meshes/visual/joint.dae" />
-        </geometry>
-      </visual>
-      <collision>
-        <origin xyz="0 0 0" rpy="0 0 0" />
-        <geometry>
-          <mesh filename="package://rik/robots/TESTy/meshes/collision/joint.stl" />
-        </geometry>
-      </collision>
-    </link>
-    <link name="testy_l5">
-      <visual>
-        <origin xyz="0 0 0" rpy="0 0 0" />
-        <geometry>
-          <mesh filename="package://rik/robots/TESTy/meshes/visual/link.dae" />
-        </geometry>
-      </visual>
-      <collision>
-        <origin xyz="0 0 0" rpy="0 0 0" />
-        <geometry>
-          <mesh filename="package://rik/robots/TESTy/meshes/collision/link.stl" />
-        </geometry>
-      </collision>
-    </link>
-    <link name="testy_j6_l">
-      <visual>
-        <origin xyz="0 0 0" rpy="0 0 0" />
-        <geometry>
-          <mesh filename="package://rik/robots/TESTy/meshes/visual/joint.dae" />
-        </geometry>
-      </visual>
-      <collision>
-        <origin xyz="0 0 0" rpy="0 0 0" />
-        <geometry>
-          <mesh filename="package://rik/robots/TESTy/meshes/collision/joint.stl" />
-        </geometry>
-      </collision>
-    </link>
-    <link name="testy_l6">
-      <visual>
-        <origin xyz="0 0 0" rpy="0 0 0" />
-        <geometry>
-          <mesh filename="package://rik/robots/TESTy/meshes/visual/link.dae" />
-        </geometry>
-      </visual>
-      <collision>
-        <origin xyz="0 0 0" rpy="0 0 0" />
-        <geometry>
-          <mesh filename="package://rik/robots/TESTy/meshes/collision/link.stl" />
-        </geometry>
-      </collision>
-    </link>
-    <link name="testy_j7_l">
-      <visual>
-        <origin xyz="0 0 0" rpy="0 0 0" />
-        <geometry>
-          <mesh filename="package://rik/robots/TESTy/meshes/visual/joint.dae" />
-        </geometry>
-      </visual>
-      <collision>
-        <origin xyz="0 0 0" rpy="0 0 0" />
-        <geometry>
-          <mesh filename="package://rik/robots/TESTy/meshes/collision/joint.stl" />
-        </geometry>
-      </collision>
-    </link>
-    <link name="testy_l7">
-      <visual>
-        <origin xyz="0 0 0" rpy="0 0 0" />
-        <geometry>
-          <mesh filename="package://rik/robots/TESTy/meshes/visual/link.dae" />
-        </geometry>
-      </visual>
-      <collision>
-        <origin xyz="0 0 0" rpy="0 0 0" />
-        <geometry>
-          <mesh filename="package://rik/robots/TESTy/meshes/collision/link.stl" />
-        </geometry>
-      </collision>
-    </link>
-    <link name="testy_j8_l">
-      <visual>
-        <origin xyz="0 0 0" rpy="0 0 0" />
-        <geometry>
-          <mesh filename="package://rik/robots/TESTy/meshes/visual/joint.dae" />
-        </geometry>
-      </visual>
-      <collision>
-        <origin xyz="0 0 0" rpy="0 0 0" />
-        <geometry>
-          <mesh filename="package://rik/robots/TESTy/meshes/collision/joint.stl" />
-        </geometry>
-      </collision>
-    </link>
-    <link name="testy_l8">
-      <visual>
-        <origin xyz="0 0 0" rpy="0 0 0" />
-        <geometry>
-          <mesh filename="package://rik/robots/TESTy/meshes/visual/link.dae" />
-        </geometry>
-      </visual>
-      <collision>
-        <origin xyz="0 0 0" rpy="0 0 0" />
-        <geometry>
-          <mesh filename="package://rik/robots/TESTy/meshes/collision/link.stl" />
-        </geometry>
-      </collision>
-    </link>
-    <link name="testy_j9_l">
-      <visual>
-        <origin xyz="0 0 0" rpy="0 0 0" />
-        <geometry>
-          <mesh filename="package://rik/robots/TESTy/meshes/visual/joint.dae" />
-        </geometry>
-      </visual>
-      <collision>
-        <origin xyz="0 0 0" rpy="0 0 0" />
-        <geometry>
-          <mesh filename="package://rik/robots/TESTy/meshes/collision/joint.stl" />
-        </geometry>
-      </collision>
-    </link>
-    <link name="testy_l9">
+    <link name="testy_1_base_link">
+      <visual>
+        <origin xyz="0 0 0" rpy="0 0 0" />
+        <geometry>
+          <mesh filename="package://rik/robots/TESTy/meshes/visual/link.dae" />
+        </geometry>
+      </visual>
+      <collision>
+        <origin xyz="0 0 0" rpy="0 0 0" />
+        <geometry>
+          <mesh filename="package://rik/robots/TESTy/meshes/collision/link.stl" />
+        </geometry>
+      </collision>
+    </link>
+    <link name="testy_1_j1_l">
+      <visual>
+        <origin xyz="0 0 0" rpy="0 0 0" />
+        <geometry>
+          <mesh filename="package://rik/robots/TESTy/meshes/visual/joint.dae" />
+        </geometry>
+      </visual>
+      <collision>
+        <origin xyz="0 0 0" rpy="0 0 0" />
+        <geometry>
+          <mesh filename="package://rik/robots/TESTy/meshes/collision/joint.stl" />
+        </geometry>
+      </collision>
+    </link>
+    <link name="testy_1_l1">
+      <visual>
+        <origin xyz="0 0 0" rpy="0 0 0" />
+        <geometry>
+          <mesh filename="package://rik/robots/TESTy/meshes/visual/link.dae" />
+        </geometry>
+      </visual>
+      <collision>
+        <origin xyz="0 0 0" rpy="0 0 0" />
+        <geometry>
+          <mesh filename="package://rik/robots/TESTy/meshes/collision/link.stl" />
+        </geometry>
+      </collision>
+    </link>
+    <link name="testy_1_j2_l">
+      <visual>
+        <origin xyz="0 0 0" rpy="0 0 0" />
+        <geometry>
+          <mesh filename="package://rik/robots/TESTy/meshes/visual/joint.dae" />
+        </geometry>
+      </visual>
+      <collision>
+        <origin xyz="0 0 0" rpy="0 0 0" />
+        <geometry>
+          <mesh filename="package://rik/robots/TESTy/meshes/collision/joint.stl" />
+        </geometry>
+      </collision>
+    </link>
+    <link name="testy_1_l2">
+      <visual>
+        <origin xyz="0 0 0" rpy="0 0 0" />
+        <geometry>
+          <mesh filename="package://rik/robots/TESTy/meshes/visual/link.dae" />
+        </geometry>
+      </visual>
+      <collision>
+        <origin xyz="0 0 0" rpy="0 0 0" />
+        <geometry>
+          <mesh filename="package://rik/robots/TESTy/meshes/collision/link.stl" />
+        </geometry>
+      </collision>
+    </link>
+    <link name="testy_1_j3_l">
+      <visual>
+        <origin xyz="0 0 0" rpy="0 0 0" />
+        <geometry>
+          <mesh filename="package://rik/robots/TESTy/meshes/visual/joint.dae" />
+        </geometry>
+      </visual>
+      <collision>
+        <origin xyz="0 0 0" rpy="0 0 0" />
+        <geometry>
+          <mesh filename="package://rik/robots/TESTy/meshes/collision/joint.stl" />
+        </geometry>
+      </collision>
+    </link>
+    <link name="testy_1_l3">
+      <visual>
+        <origin xyz="0 0 0" rpy="0 0 0" />
+        <geometry>
+          <mesh filename="package://rik/robots/TESTy/meshes/visual/link.dae" />
+        </geometry>
+      </visual>
+      <collision>
+        <origin xyz="0 0 0" rpy="0 0 0" />
+        <geometry>
+          <mesh filename="package://rik/robots/TESTy/meshes/collision/link.stl" />
+        </geometry>
+      </collision>
+    </link>
+    <link name="testy_1_j4_l">
+      <visual>
+        <origin xyz="0 0 0" rpy="0 0 0" />
+        <geometry>
+          <mesh filename="package://rik/robots/TESTy/meshes/visual/joint.dae" />
+        </geometry>
+      </visual>
+      <collision>
+        <origin xyz="0 0 0" rpy="0 0 0" />
+        <geometry>
+          <mesh filename="package://rik/robots/TESTy/meshes/collision/joint.stl" />
+        </geometry>
+      </collision>
+    </link>
+    <link name="testy_1_l4">
+      <visual>
+        <origin xyz="0 0 0" rpy="0 0 0" />
+        <geometry>
+          <mesh filename="package://rik/robots/TESTy/meshes/visual/link.dae" />
+        </geometry>
+      </visual>
+      <collision>
+        <origin xyz="0 0 0" rpy="0 0 0" />
+        <geometry>
+          <mesh filename="package://rik/robots/TESTy/meshes/collision/link.stl" />
+        </geometry>
+      </collision>
+    </link>
+    <link name="testy_1_j5_l">
+      <visual>
+        <origin xyz="0 0 0" rpy="0 0 0" />
+        <geometry>
+          <mesh filename="package://rik/robots/TESTy/meshes/visual/joint.dae" />
+        </geometry>
+      </visual>
+      <collision>
+        <origin xyz="0 0 0" rpy="0 0 0" />
+        <geometry>
+          <mesh filename="package://rik/robots/TESTy/meshes/collision/joint.stl" />
+        </geometry>
+      </collision>
+    </link>
+    <link name="testy_1_l5">
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